File: la-caja/pruebas/prueba3-reloj/La caja/La caja.kicad_sch (KiCad schematic)
At the start: 1 part, among them U1 NodeMCU1.0(ESP-12E)

Commit message: Kicad testing worked!
Parts:
- removed U1: NodeMCU1.0(ESP-12E), symbol ESP8266:NodeMCU1.0(ESP-12E)
Other:
- added sheet Prueba_1 (Prueba_1.kicad_sch)
- added sheet Prueba_2 (Prueba_2.kicad_sch)
- added sheet Prueba_3 (Prueba_3.kicad_sch)
- added sheet Prueba_4 (Prueba_4.kicad_sch)
- added sheet Prueba_5 (Prueba_5.kicad_sch)
- company: RhylooSolutions -> Proyecto la Caja
- title: Testting de esquematicos -> Testing de esquematicos
