File: la-caja/pruebas/jorge/prueba3-reloj/La caja/Prueba_1.kicad_sch (KiCad schematic)
At the start: 1 part

Commit message: Kicad testin some new features
Parts:
- added 96BB2-006-F?: 4x4_Keypad, symbol KEYPAD:4x4_Keypad
Changed lines of the file:
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@@
     (pin "9")
+  )
+  (symbol (lib_id "KEYPAD:4x4_Keypad") (at 66.04 118.11 270) (unit 1)
+    (in_bom yes) (on_board yes) (fields_autoplaced)
+    (property "Reference" "96BB2-006-F?" (id 0) (at 66.675 92.71 90)
+      (effects (font (size 1.524 1.524)))
+    )
+    (property "Value" "4x4_Keypad" (id 1) (at 66.675 96.52 90)
+      (effects (font (size 1.524 1.524)))
+    )
+    (property "Footprint" "" (id 2) (at 66.04 118.11 0)
+      (effects (font (size 1.524 1.524)))
+    )
+    (property "Datasheet" "" (id 3) (at 66.04 118.11 0)
+      (effects (font (size 1.524 1.524)))
+    )
+    (pin "~")
+    (pin "~")
+    (pin "~")
+    (pin "~")
+    (pin "~")
+    (pin "~")
+    (pin "~")
+    (pin "~")
   )
   (sheet_instances
