File: la-caja/kicad/Prueba_3.kicad_sch (KiCad schematic)
At the start: 4 parts, among them U1 ADS1015IDGS, U1 Joystick

Commit message: Esquematico actualizado, nuevo símbolo para numpad
Parts:
- renumbered Cara003 to Cara3
Changed lines of the file:
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@@
   (symbol (lib_id "ESP8266:NodeMCU1.0(ESP-12E)") (at 81.28 137.16 0) (unit 1)
     (in_bom yes) (on_board yes)
-    (property "Reference" "Cara003" (id 0) (at 81.28 109.22 0)
+    (property "Reference" "Cara3" (id 0) (at 81.28 109.22 0)
       (effects (font (size 1.524 1.524)))
     )
