File: la-caja/kicad/Prueba_4.kicad_sch (KiCad schematic)
At the start: 1 part

Commit message: Cambios en KiCAD
Parts:
- removed PRUEBA4: NodeMCU1.0(ESP-12E), symbol ESP8266:NodeMCU1.0(ESP-12E)
Changed lines of the file:
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@@
     (company "Proyecto la Caja")
-  )
-  (wire (pts (xy 49.53 62.23) (xy 64.77 62.23))
-    (stroke (width 0) (type default) (color 0 0 0 0))
-  )
-  (wire (pts (xy 49.53 59.69) (xy 64.77 59.69))
-    (stroke (width 0) (type default) (color 0 0 0 0))
-  )
-  (hierarchical_label "GND" (shape input) (at 49.53 59.69 180)
-    (effects (font (size 1.27 1.27)) (justify right))
-  )
-  (hierarchical_label "VCC" (shape input) (at 49.53 62.23 180)
-    (effects (font (size 1.27 1.27)) (justify right))
-  )
-  (symbol (lib_id "ESP8266:NodeMCU1.0(ESP-12E)") (at 85.09 44.45 0) (unit 1)
-    (in_bom yes) (on_board yes)
-    (property "Reference" "PRUEBA4" (id 0) (at 85.09 16.51 0)
-      (effects (font (size 1.524 1.524)))
-    )
-    (property "Value" "NodeMCU1.0(ESP-12E)" (id 1) (at 85.09 20.32 0)
-      (effects (font (size 1.524 1.524)))
-    )
-    (property "Footprint" "" (id 2) (at 69.85 66.04 0)
-      (effects (font (size 1.524 1.524)))
-    )
-    (property "Datasheet" "https://www.esploradores.com/wp-content/uploads/2019/11/PINOUT-NodeMCU_1.0-V2-2_2.jpg" (id 3) (at 85.09 69.85 0)
-      (effects (font (size 1.524 1.524)))
-    )
-    (property "Precio" "10€" (id 4) (at 85.09 44.45 0)
-      (effects (font (size 1.27 1.27)) hide)
-    )
-    (pin "1")
-    (pin "10")
-    (pin "11")
-    (pin "12")
-    (pin "13")
-    (pin "14")
-    (pin "15")
-    (pin "16")
-    (pin "17")
-    (pin "18")
-    (pin "19")
-    (pin "2")
-    (pin "20")
-    (pin "21")
-    (pin "22")
-    (pin "23")
-    (pin "24")
-    (pin "25")
-    (pin "26")
-    (pin "27")
-    (pin "28")
-    (pin "29")
-    (pin "3")
-    (pin "30")
-    (pin "4")
-    (pin "5")
-    (pin "6")
-    (pin "7")
-    (pin "8")
-    (pin "9")
   )
   (sheet_instances
